File: sm_charlieplex_rgb_battery.kicad_pcb (KiCad board)
At the start: 2 copper layers, 12 x 12 mm, 12 parts, among them SW1 SW_Push, U1 ATtiny10-TS

Commit message: Finish routing
Parts:
- moved R4 0.84 mm to (171.9, 106.3), turned to 270 degrees
- moved SW1 0.09 mm to (165.8, 105.8)
Routing:
- net Net-(D1-Pad1): track 1.60 -> 26.3 mm, vias 0 -> 4
- net Net-(D1-Pad3): track 5.06 -> 29.1 mm, vias 0 -> 5
- net Net-(D1-Pad4): track 3.91 -> 25.9 mm, vias 0 -> 4
- net Net-(D1-Pad2): track 4.57 -> 20.7 mm
- net /+3V: track 18.8 -> 8.76 mm
- net Net-(C1-Pad1): track 12.6 -> 15.4 mm
- net Net-(R1-Pad2): track 2.56 -> 3.07 mm
- removed copper zone on B.Cu, net (none)
- removed copper zone on F.Cu, net (none)

Commit message: Bump version on board
Other:
- board text added: "WM v2.0.0 09/25/19"
- board text removed: "WM v2.0.0 09/17/19"
Changed lines of the file:
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@@
   )
   (setup
-    (last_trace_width 0.2)
+    (last_trace_width 0.25)
     (user_trace_width 0.2)
     (trace_clearance 0.2)
@@
     )
   )
-  (gr_text "WM v2.0.0\n09/17/19" (at 171.196 106.7 180) (layer B.SilkS)
+  (gr_text "WM v2.0.0\n09/25/19" (at 171.196 106.7 180) (layer B.SilkS)
     (effects (font (size 0.5 0.5) (thickness 0.125)) (justify mirror))
   )
